File: kicad/buck_3a_v4.sch (KiCad schematic (older format))
At the start: 26 parts, among them J1 LED+, J2 LED-, J3 Conn_01x04, J4 Conn_01x02, J5 Conn_01x06, Q1 BSC050N03, U1 MAX16820ATT, U2 ATtiny45-20SU

Commit message: mech/ Lampengehäuse getauscht zu Variante mit O-Ring
kicad/
Neue Version mit besserem Layout
Neue JLC Daten
Parts:
- removed J4: Conn_01x02, Connector_PinHeader_2.00mm:PinHeader_1x02_P2.00mm_Vertical, symbol Connector_Generic:Conn_01x02
- added C7: 22u0/16V, Capacitor_SMD:C_0805_2012Metric, symbol Device:C
- added R8: CMFB103F3950FANT, Resistor_SMD:R_0805_2012Metric, symbol Device:R
- C1: value 22u0 -> 100u/16V; footprint Capacitor_SMD:C_0805_2012Metric -> Capacitor_SMD:C_1210_3225Metric; LCSC C45783 -> C90143
- C3: value 22u0 -> DNP; LCSC C45783 -> (none)
- C4: value 22u0 -> 22u0/16V
- C6: LCSC (none) -> C1744
- D1: value PDS1040 -> SS54; footprint Diode_SMD:D_PowerDI-5 -> Diode_SMD:D_SMA
- L1: value WE7447714100 -> MWSA0603-100MT; footprint Inductor_SMD:L_10.4x10.4_H4.8 -> Inductor_SMD:L_Sumida_CDMC6D28_7.25x6.5mm
- Q1: value BSC050N03 -> BSC022N04LSATMA; LCSC C139521 -> C148266
Connections:
- wire segments 67 -> 72
Changed lines of the file:
@@
 P 4350 2600
 F 0 "L1" V 4540 2600 50  0000 C CNN
-F 1 "WE7447714100" V 4449 2600 50  0000 C CNN
-F 2 "Inductor_SMD:L_10.4x10.4_H4.8" H 4350 2600 50  0001 C CNN
+F 1 "MWSA0603-100MT" V 4449 2600 50  0000 C CNN
+F 2 "Inductor_SMD:L_Sumida_CDMC6D28_7.25x6.5mm" H 4350 2600 50  0001 C CNN
 F 3 "~" H 4350 2600 50  0001 C CNN
 F 4 "C132141" V 4350 2600 50  0001 C CNN "LCSC"
@@
 P 4800 3800
 F 0 "Q1" H 5005 3846 50  0000 L CNN
-F 1 "BSC050N03" H 5005 3755 50  0000 L CNN
+F 1 "BSC022N04LSATMA" H 5005 3755 50  0000 L CNN
 F 2 "Package_TO_SOT_SMD:TDSON-8-1" H 5000 3725 50  0001 L CIN
 F 3 "http://www.infineon.com/dgdl/Infineon-BSC040N08NS5-DS-v02_00-EN.pdf?fileId=5546d4624ad04ef9014ae3065a7e2a05" V 4800 3800 50  0001 L CNN
-F 4 "C139521" H 4800 3800 50  0001 C CNN "LCSC"
+F 4 " C148266" H 4800 3800 50  0001 C CNN "LCSC"
 	1    4800 3800
 	1    0    0    -1
@@
 P 3400 2250
 F 0 "D1" H 3400 2467 50  0000 C CNN
-F 1 "PDS1040" H 3400 2376 50  0000 C CNN
-F 2 "Diode_SMD:D_PowerDI-5" H 3400 2250 50  0001 C CNN
+F 1 "SS54" H 3400 2376 50  0000 C CNN
+F 2 "Diode_SMD:D_SMA" H 3400 2250 50  0001 C CNN
 F 3 "~" H 3400 2250 50  0001 C CNN
 F 4 "C22452" H 3400 2250 50  0001 C CNN "LCSC"
@@
 $EndComp
 $Comp
-L Connector_Generic:Conn_01x02 J4
-U 1 1 5F9D60F0
-P 8450 4300
-F 0 "J4" H 8530 4292 50  0000 L CNN
-F 1 "Conn_01x02" H 8530 4201 50  0000 L CNN
-F 2 "Connector_PinHeader_2.00mm:PinHeader_1x02_P2.00mm_Vertical" H 8450 4300 50  0001 C CNN
-F 3 "~" H 8450 4300 50  0001 C CNN
-	1    8450 4300
-	1    0    0    -1
-$EndComp
-$Comp
 L Device:R R7
 U 1 1 5F9DA62A
@@
 P 6600 2600
 F 0 "C4" H 6715 2646 50  0000 L CNN
-F 1 "22u0" H 6715 2555 50  0000 L CNN
+F 1 "22u0/16V" H 6715 2555 50  0000 L CNN
 F 2 "Capacitor_SMD:C_0805_2012Metric" H 6638 2450 50  0001 C CNN
 F 3 "~" H 6600 2600 50  0001 C CNN
 F 4 "C45783" H 6600 2600 50  0001 C CNN "LCSC"
 	1    6600 2600
-	1    0    0    -1
-$EndComp
-$Comp
-L Device:C C3
-U 1 1 5F9EC8A9
-P 2900 2950
-F 0 "C3" H 3015 2996 50  0000 L CNN
-F 1 "22u0" H 3015 2905 50  0000 L CNN
-F 2 "Capacitor_SMD:C_0805_2012Metric" H 2938 2800 50  0001 C CNN
-F 3 "~" H 2900 2950 50  0001 C CNN
-F 4 "C45783" H 2900 2950 50  0001 C CNN "LCSC"
-	1    2900 2950
 	1    0    0    -1
 $EndComp
@@
 	2600 2600 2650 2600
 Wire Wire Line
-	3750 2600 4200 2600
+	3750 2600 3850 2600
 Wire Wire Line
 	4500 2600 4900 2600
@@
 $EndComp
 Wire Wire Line
-	4150 3600 4300 3600
-Wire Wire Line
-	2900 2600 2900 2800
+	4150 3600 4250 3600
 Connection ~ 2900 2600
 Wire Wire Line
 	2900 2600 3050 2600
-$Comp
-L power:GND #PWR0103
-U 1 1 5FA20125
-P 2900 3250
-F 0 "#PWR0103" H 2900 3000 50  0001 C CNN
-F 1 "GND" H 2905 3077 50  0000 C CNN
-F 2 "" H 2900 3250 50  0001 C CNN
-F 3 "" H 2900 3250 50  0001 C CNN
-	1    2900 3250
-	1    0    0    -1
-$EndComp
-Wire Wire Line
-	2900 3100 2900 3250
 Wire Wire Line
 	2650 2600 2650 3800
@@
 	1    0    0    -1
 $EndComp
-$Comp
-L Device:C C1
-U 1 1 5F9EA3C0
-P 1350 2950
-F 0 "C1" H 1465 2996 50  0000 L CNN
-F 1 "22u0" H 1465 2905 50  0000 L CNN
-F 2 "Capacitor_SMD:C_0805_2012Metric" H 1388 2800 50  0001 C CNN
-F 3 "~" H 1350 2950 50  0001 C CNN
-F 4 "C45783" H 1350 2950 50  0001 C CNN "LCSC"
-	1    1350 2950
-	1    0    0    -1
-$EndComp
 Wire Wire Line
 	7000 2450 7000 2300
@@
 	8050 4250 8050 4300
 Wire Wire Line
-	8050 4300 8250 4300
+	8050 4300 8050 4400
 $Comp
 L power:GND #PWR0116
 U 1 1 5FA9B588
-P 8250 4400
-F 0 "#PWR0116" H 8250 4150 50  0001 C CNN
-F 1 "GND" H 8255 4227 50  0000 C CNN
-F 2 "" H 8250 4400 50  0001 C CNN
-F 3 "" H 8250 4400 50  0001 C CNN
-	1    8250 4400
+P 8050 4700
+F 0 "#PWR0116" H 8050 4450 50  0001 C CNN
+F 1 "GND" H 8055 4527 50  0000 C CNN
+F 2 "" H 8050 4700 50  0001 C CNN
+F 3 "" H 8050 4700 50  0001 C CNN
+	1    8050 4700
 	1    0    0    -1
 $EndComp
@@
 F 2 "Capacitor_SMD:C_0805_2012Metric" H 7238 4400 50  0001 C CNN
 F 3 "~" H 7200 4550 50  0001 C CNN
+F 4 "C1744" H 7200 4550 50  0001 C CNN "LCSC"
 	1    7200 4550
 	1    0    0    -1
@@
 	7200 4700 6800 4700
 Connection ~ 6800 4700
+$Comp
+L Device:C C1
+U 1 1 6079EE15
+P 1350 2950
+F 0 "C1" H 1465 2996 50  0000 L CNN
+F 1 "100u/16V" H 1465 2905 50  0000 L CNN
+F 2 "Capacitor_SMD:C_1210_3225Metric" H 1388 2800 50  0001 C CNN
+F 3 "~" H 1350 2950 50  0001 C CNN
+F 4 "C90143" H 1350 2950 50  0001 C CNN "LCSC"
+	1    1350 2950
+	1    0    0    -1
+$EndComp
+$Comp
+L Device:C C3
+U 1 1 607A3389
+P 3400 3050
+F 0 "C3" V 3148 3050 50  0000 C CNN
+F 1 "DNP" V 3239 3050 50  0000 C CNN
+F 2 "Capacitor_SMD:C_0805_2012Metric" H 3438 2900 50  0001 C CNN
+F 3 "~" H 3400 3050 50  0001 C CNN
+	1    3400 3050
+	0    1    1    0
+$EndComp
+Wire Wire Line
+	2900 3050 3250 3050
+Wire Wire Line
+	2900 2600 2900 3050
+Wire Wire Line
+	3550 3050 3850 3050
+Wire Wire Line
+	3850 3050 3850 2600
+Connection ~ 3850 2600
+Wire Wire Line
+	3850 2600 4200 2600
+$Comp
+L Device:C C7
+U 1 1 607A7D2F
+P 4250 4050
+F 0 "C7" H 4365 4096 50  0000 L CNN
+F 1 "22u0/16V" H 4365 4005 50  0000 L CNN
+F 2 "Capacitor_SMD:C_0805_2012Metric" H 4288 3900 50  0001 C CNN
+F 3 "~" H 4250 4050 50  0001 C CNN
+F 4 "C45783" H 4250 4050 50  0001 C CNN "LCSC"
+	1    4250 4050
+	1    0    0    -1
+$EndComp
+Wire Wire Line
+	4250 3900 4250 3600
+Connection ~ 4250 3600
+Wire Wire Line
+	4250 3600 4300 3600
+$Comp
+L power:GND #PWR0103
+U 1 1 607AA26C
+P 4250 4200
+F 0 "#PWR0103" H 4250 3950 50  0001 C CNN
+F 1 "GND" H 4255 4027 50  0000 C CNN
+F 2 "" H 4250 4200 50  0001 C CNN
+F 3 "" H 4250 4200 50  0001 C CNN
+	1    4250 4200
+	1    0    0    -1
+$EndComp
+$Comp
+L Device:R R8
+U 1 1 6078CC24
+P 8050 4550
+F 0 "R8" H 8120 4596 50  0000 L CNN
+F 1 "CMFB103F3950FANT" H 8120 4505 50  0000 L CNN
+F 2 "Resistor_SMD:R_0805_2012Metric" V 7980 4550 50  0001 C CNN
+F 3 "~" H 8050 4550 50  0001 C CNN
+F 4 "C51597" H 8050 4550 50  0001 C CNN "LCSC"
+	1    8050 4550
+	1    0    0    -1
+$EndComp
 $EndSCHEMATC
