File: kicad/buck_3a_v4.kicad_pcb (KiCad board)
At the start: 2 copper layers, 44 x 44 mm, 26 parts, among them J1 LED+, J2 LED-, J3 Conn_01x04, J4 Conn_01x02, J5 Conn_01x06, Q1 BSC050N03, U1 MAX16820ATT, U2 ATtiny45-20SU

Commit message: mech/ Lampengehäuse getauscht zu Variante mit O-Ring
kicad/
Neue Version mit besserem Layout
Neue JLC Daten
Parts:
- removed J4: Conn_01x02, Connector_PinHeader_2.00mm:PinHeader_1x02_P2.00mm_Vertical
- added C7: 22u0/16V, Capacitor_SMD:C_0805_2012Metric, F.Cu at (58.7, 34.1)
- added R8: CMFB103F3950FANT, Resistor_SMD:R_0805_2012Metric, F.Cu at (40.2, 62.6)
- C1: value 22u0 -> 100u/16V; footprint Capacitor_SMD:C_0805_2012Metric -> Capacitor_SMD:C_1210_3225Metric
- C3: value 22u0 -> DNP
- C4: value 22u0 -> 22u0/16V
- D1: value PDS1040 -> SS54; footprint Diode_SMD:D_PowerDI-5 -> Diode_SMD:D_SMA
- L1: value WE7447714100 -> MWSA0603-100MT; footprint Inductor_SMD:L_10.4x10.4_H4.8 -> Inductor_SMD:L_Sumida_CDMC6D28_7.25x6.5mm
- Q1: value BSC050N03 -> BSC022N04LSATMA
- moved C3 9.23 mm to (57.0, 45.7), turned to 0 degrees
- moved Q1 7.40 mm to (44.6, 40.3), turned to 90 degrees
- moved C1 7.40 mm to (51.4, 42.8)
- moved C2 6.83 mm to (51.6, 39.9)
- moved D1 5.50 mm to (51.4, 36.9)
- moved U1 3.76 mm to (58.6, 37.8)
- moved L1 3.28 mm to (37.8, 40.7), turned to 90 degrees
- moved R1 1.73 mm to (58.2, 42.4)
- renumbered J1 to LED+, J2 to LED-
Connections:
- C3 pad 2: GND -> Net-(C3-Pad2)
- L1 pad 1: Net-(J2-Pad1) -> Net-(C3-Pad1)
- LED+ pad 1: Net-(C3-Pad1) -> Net-(C3-Pad2)
- LED- pad 1: Net-(J2-Pad1) -> Net-(C3-Pad1)
- R1 pad 1: Net-(C3-Pad1) -> Net-(C3-Pad2)
- U1 pad 2: Net-(C3-Pad1) -> Net-(C3-Pad2)
Routing:
- net VCC: track 33.2 -> 23.2 mm
- net Net-(C3-Pad1): track 10.0 -> 17.8 mm, vias 0 -> 1
- net GND: track 19.1 -> 12.0 mm, vias 16 -> 15
- net Net-(Q1-Pad4): track 9.44 -> 16.4 mm, vias 0 -> 2
- net Net-(C3-Pad2): track 0.00 -> 5.38 mm
- net +5V: track 88.6 -> 92.1 mm
- net /PWM: track 39.8 -> 36.8 mm
- net /TMESS: track 7.13 -> 6.18 mm
- net /MODE: track 27.2 -> 27.5 mm, vias 0 -> 2
- added copper zone on F.Cu, net Net-(C3-Pad2)
- removed copper zone on F.Cu, net Net-(J2-Pad1)
Other:
- board text added: "LED v4.2 GS 2021"
- board text removed: "LED v4.1 GS 2020"
