File: kicad/buck_3a_v4.kicad_pcb (KiCad board)
At the start: 2 copper layers, 44 x 44 mm, 27 parts, among them J3 Conn_01x04, J5 Conn_01x06, Q1 BSC022N04LSATMA, U1 MAX16820ATT, U2 ATtiny45-20SU

Commit message: Save V4.3
Other:
- net class Default removed
- board text added: "LED v4.3 GS 2021"
- board text removed: "LED v4.2 GS 2021"
