File: kicad/batteriedeckel/batteriedeckel/batteriedeckel.kicad_sch (KiCad schematic)
At the start: 7 parts, among them J1 Conn_01x03

Commit message: save
Parts:
- BAT+1: renamed from TP1; footprint TestPoint:TestPoint_THTPad_D4.0mm_Drill2.0mm -> TestPoint:TestPoint_THTPad_D5.0mm_Drill3.0mm
- BAT-1: renamed from TP2; footprint TestPoint:TestPoint_THTPad_D4.0mm_Drill2.0mm -> TestPoint:TestPoint_THTPad_D5.0mm_Drill3.0mm
- SW+1: renamed from TP3; footprint TestPoint:TestPoint_THTPad_D4.0mm_Drill2.0mm -> TestPoint:TestPoint_THTPad_D5.0mm_Drill3.0mm
- SW-1: renamed from TP4; footprint TestPoint:TestPoint_THTPad_D4.0mm_Drill2.0mm -> TestPoint:TestPoint_THTPad_D5.0mm_Drill3.0mm
Changed lines of the file:
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@@
   (symbol (lib_id "Connector:TestPoint") (at 97.155 86.995 90) (unit 1)
     (in_bom yes) (on_board yes) (fields_autoplaced)
-    (property "Reference" "TP4" (id 0) (at 93.853 82.6602 90))
+    (property "Reference" "SW-1" (id 0) (at 93.853 82.6602 90))
     (property "Value" "SW-" (id 1) (at 93.853 85.1971 90))
-    (property "Footprint" "TestPoint:TestPoint_THTPad_D4.0mm_Drill2.0mm" (id 2) (at 97.155 81.915 0)
+    (property "Footprint" "TestPoint:TestPoint_THTPad_D5.0mm_Drill3.0mm" (id 2) (at 97.155 81.915 0)
       (effects (font (size 1.27 1.27)) hide)
     )
@@
   (symbol (lib_id "Connector:TestPoint") (at 97.155 80.645 90) (unit 1)
     (in_bom yes) (on_board yes) (fields_autoplaced)
-    (property "Reference" "TP2" (id 0) (at 93.853 76.3102 90))
+    (property "Reference" "BAT-1" (id 0) (at 93.853 76.3102 90))
     (property "Value" "BAT-" (id 1) (at 93.853 78.8471 90))
-    (property "Footprint" "TestPoint:TestPoint_THTPad_D4.0mm_Drill2.0mm" (id 2) (at 97.155 75.565 0)
+    (property "Footprint" "TestPoint:TestPoint_THTPad_D5.0mm_Drill3.0mm" (id 2) (at 97.155 75.565 0)
       (effects (font (size 1.27 1.27)) hide)
     )
@@
   (symbol (lib_id "Connector:TestPoint") (at 97.155 71.755 90) (unit 1)
     (in_bom yes) (on_board yes) (fields_autoplaced)
-    (property "Reference" "TP1" (id 0) (at 93.853 67.4202 90))
+    (property "Reference" "BAT+1" (id 0) (at 93.853 67.4202 90))
     (property "Value" "BAT+" (id 1) (at 93.853 69.9571 90))
-    (property "Footprint" "TestPoint:TestPoint_THTPad_D4.0mm_Drill2.0mm" (id 2) (at 97.155 66.675 0)
+    (property "Footprint" "TestPoint:TestPoint_THTPad_D5.0mm_Drill3.0mm" (id 2) (at 97.155 66.675 0)
       (effects (font (size 1.27 1.27)) hide)
     )
@@
   (symbol (lib_id "Connector:TestPoint") (at 96.52 94.615 90) (unit 1)
     (in_bom yes) (on_board yes) (fields_autoplaced)
-    (property "Reference" "TP3" (id 0) (at 93.218 90.2802 90))
+    (property "Reference" "SW+1" (id 0) (at 93.218 90.2802 90))
     (property "Value" "SW+" (id 1) (at 93.218 92.8171 90))
-    (property "Footprint" "TestPoint:TestPoint_THTPad_D4.0mm_Drill2.0mm" (id 2) (at 96.52 89.535 0)
+    (property "Footprint" "TestPoint:TestPoint_THTPad_D5.0mm_Drill3.0mm" (id 2) (at 96.52 89.535 0)
       (effects (font (size 1.27 1.27)) hide)
     )
@@
   )
   (symbol_instances
+    (path "/54cd7fa4-6408-45bc-b94e-25c077756cf9"
+      (reference "BAT+1") (unit 1) (value "BAT+") (footprint "TestPoint:TestPoint_THTPad_D5.0mm_Drill3.0mm")
+    )
+    (path "/464be180-2649-40a5-986a-553388dceed3"
+      (reference "BAT-1") (unit 1) (value "BAT-") (footprint "TestPoint:TestPoint_THTPad_D5.0mm_Drill3.0mm")
+    )
     (path "/31544892-8ec4-47ce-b873-1f2750fb72dd"
       (reference "H1") (unit 1) (value "MountingHole") (footprint "MountingHole:MountingHole_3.2mm_M3_DIN965")
@@
       (reference "J1") (unit 1) (value "Conn_01x03") (footprint "Connector_PinSocket_2.00mm:PinSocket_1x03_P2.00mm_Vertical_SMD_Pin1Left")
     )
-    (path "/54cd7fa4-6408-45bc-b94e-25c077756cf9"
-      (reference "TP1") (unit 1) (value "BAT+") (footprint "TestPoint:TestPoint_THTPad_D4.0mm_Drill2.0mm")
-    )
-    (path "/464be180-2649-40a5-986a-553388dceed3"
-      (reference "TP2") (unit 1) (value "BAT-") (footprint "TestPoint:TestPoint_THTPad_D4.0mm_Drill2.0mm")
-    )
     (path "/a95940ed-da1c-4634-9ca1-d2cdfdc2c676"
-      (reference "TP3") (unit 1) (value "SW+") (footprint "TestPoint:TestPoint_THTPad_D4.0mm_Drill2.0mm")
+      (reference "SW+1") (unit 1) (value "SW+") (footprint "TestPoint:TestPoint_THTPad_D5.0mm_Drill3.0mm")
     )
     (path "/3af06d96-7f67-4ae4-b571-d05d98fbc8a6"
-      (reference "TP4") (unit 1) (value "SW-") (footprint "TestPoint:TestPoint_THTPad_D4.0mm_Drill2.0mm")
+      (reference "SW-1") (unit 1) (value "SW-") (footprint "TestPoint:TestPoint_THTPad_D5.0mm_Drill3.0mm")
     )
   )
