File: kicad/batteriedeckel/batteriedeckel/batteriedeckel.kicad_pcb (KiCad board)
At the start: 2 copper layers, 44 x 44 mm, 7 parts, among them J1 Conn_01x03

Commit message: save
Parts:
- BAT+, BAT-, SW+, SW-: footprint TestPoint:TestPoint_THTPad_D4.0mm_Drill2.0mm -> TestPoint:TestPoint_THTPad_D5.0mm_Drill3.0mm
- moved J1 2.30 mm to (97.7, 100.0), turned to 0 degrees
- moved BAT- 2.24 mm to (102.0, 102.0)
- moved H1 0.50 mm to (100.0, 82.0)
- moved H2 0.50 mm to (100.0, 118.0)
Routing:
- net /MODE: track 15.9 -> 12.1 mm
Changed lines of the file:
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@@
   (net 3 "/MODE")
   (footprint "MountingHole:MountingHole_3.2mm_M3_DIN965" (layer "F.Cu")
-    (at 100 117.5)
+    (at 100 118)
     (descr "Mounting Hole 3.2mm, no annular, M3, DIN965")
     (tags "mounting hole 3.2mm no annular m3 din965")
@@
   )
   (footprint "MountingHole:MountingHole_3.2mm_M3_DIN965" (layer "F.Cu")
-    (at 100 82.5)
+    (at 100 82)
     (descr "Mounting Hole 3.2mm, no annular, M3, DIN965")
     (tags "mounting hole 3.2mm no annular m3 din965")
@@
     (pad "" np_thru_hole circle (at 0 0) (size 3.2 3.2) (drill 3.2) (layers *.Cu *.Mask))
   )
-  (footprint "TestPoint:TestPoint_THTPad_D4.0mm_Drill2.0mm" (layer "F.Cu")
+  (footprint "TestPoint:TestPoint_THTPad_D5.0mm_Drill3.0mm" (layer "F.Cu")
     (at 92.75 87.443)
     (descr "THT pad as test Point, diameter 4.0mm, hole diameter 2.0mm")
@@
     (property "Sheetfile" "batteriedeckel.kicad_sch")
     (property "Sheetname" "")
-    (attr exclude_from_pos_files)
-    (fp_text reference "BAT+" (at -4.866 -0.067) (layer "F.SilkS")
+    (attr exclude_from_pos_files exclude_from_bom)
+    (fp_text reference "BAT+" (at 0 -2.898) (layer "F.SilkS")
       (effects (font (size 1 1) (thickness 0.15)))
     )
@@
       (effects (font (size 1 1) (thickness 0.15)))
     )
-    (fp_circle (center 0 0) (end 0 2.25) (layer "F.SilkS") (width 0.12) (fill none))
-    (fp_circle (center 0 0) (end 2.5 0) (layer "F.CrtYd") (width 0.05) (fill none))
-    (pad "1" thru_hole circle (at 0 0) (size 4 4) (drill 2) (layers *.Cu *.Mask)
+    (fp_circle (center 0 0) (end 2.5 0) (layer "F.SilkS") (width 0.12) (fill none))
+    (fp_circle (center 0 0) (end 3 0) (layer "F.CrtYd") (width 0.05) (fill none))
+    (pad "1" thru_hole circle (at 0 0) (size 5 5) (drill 3) (layers *.Cu *.Mask)
       (net 1 "/BAT+") (pinfunction "1") (pintype "passive"))
   )
-  (footprint "TestPoint:TestPoint_THTPad_D4.0mm_Drill2.0mm" (layer "F.Cu")
+  (footprint "TestPoint:TestPoint_THTPad_D5.0mm_Drill3.0mm" (layer "F.Cu")
     (at 114.5 100)
     (descr "THT pad as test Point, diameter 4.0mm, hole diameter 2.0mm")
@@
     (property "Sheetfile" "batteriedeckel.kicad_sch")
     (property "Sheetname" "")
-    (attr exclude_from_pos_files)
-    (fp_text reference "SW-" (at 4.626 0.076) (layer "F.SilkS")
-      (effects (font (size 1 1) (thickness 0.15)))
-    )
-    (fp_text value "SW-" (at 4.626 0.076) (layer "F.Fab")
-      (effects (font (size 1 1) (thickness 0.15)))
-    )
-    (fp_text user "${REFERENCE}" (at 0 -2.9) (layer "F.Fab")
-      (effects (font (size 1 1) (thickness 0.15)))
-    )
-    (fp_circle (center 0 0) (end 0 2.25) (layer "F.SilkS") (width 0.12) (fill none))
-    (fp_circle (center 0 0) (end 2.5 0) (layer "F.CrtYd") (width 0.05) (fill none))
-    (pad "1" thru_hole circle (at 0 0) (size 4 4) (drill 2) (layers *.Cu *.Mask)
+    (attr exclude_from_pos_files exclude_from_bom)
+    (fp_text reference "SW-" (at 0 -2.898) (layer "F.SilkS")
+      (effects (font (size 1 1) (thickness 0.15)))
+    )
+    (fp_text value "SW-" (at 0 3.1) (layer "F.Fab")
+      (effects (font (size 1 1) (thickness 0.15)))
+    )
+    (fp_text user "${REFERENCE}" (at 0 -2.9) (layer "F.Fab")
+      (effects (font (size 1 1) (thickness 0.15)))
+    )
+    (fp_circle (center 0 0) (end 2.5 0) (layer "F.SilkS") (width 0.12) (fill none))
+    (fp_circle (center 0 0) (end 3 0) (layer "F.CrtYd") (width 0.05) (fill none))
+    (pad "1" thru_hole circle (at 0 0) (size 5 5) (drill 3) (layers *.Cu *.Mask)
       (net 2 "/GND") (pinfunction "1") (pintype "passive"))
   )
-  (footprint "TestPoint:TestPoint_THTPad_D4.0mm_Drill2.0mm" (layer "F.Cu")
-    (at 103 104)
-    (descr "THT pad as test Point, diameter 4.0mm, hole diameter 2.0mm")
-    (tags "test point THT pad")
-    (property "Sheetfile" "batteriedeckel.kicad_sch")
-    (property "Sheetname" "")
-    (attr exclude_from_pos_files)
-    (fp_text reference "BAT-" (at 4.95 0.394) (layer "F.SilkS")
+  (footprint "TestPoint:TestPoint_THTPad_D5.0mm_Drill3.0mm" (layer "F.Cu")
+    (at 102 102)
+    (descr "THT pad as test Point, diameter 4.0mm, hole diameter 2.0mm")
+    (tags "test point THT pad")
+    (property "Sheetfile" "batteriedeckel.kicad_sch")
+    (property "Sheetname" "")
+    (attr exclude_from_pos_files exclude_from_bom)
+    (fp_text reference "BAT-" (at 0 -2.898) (layer "F.SilkS")
       (effects (font (size 1 1) (thickness 0.15)))
     )
@@
       (effects (font (size 1 1) (thickness 0.15)))
     )
-    (fp_circle (center 0 0) (end 0 2.25) (layer "F.SilkS") (width 0.12) (fill none))
-    (fp_circle (center 0 0) (end 2.5 0) (layer "F.CrtYd") (width 0.05) (fill none))
-    (pad "1" thru_hole circle (at 0 0) (size 4 4) (drill 2) (layers *.Cu *.Mask)
+    (fp_circle (center 0 0) (end 2.5 0) (layer "F.SilkS") (width 0.12) (fill none))
+    (fp_circle (center 0 0) (end 3 0) (layer "F.CrtYd") (width 0.05) (fill none))
+    (pad "1" thru_hole circle (at 0 0) (size 5 5) (drill 3) (layers *.Cu *.Mask)
       (net 2 "/GND") (pinfunction "1") (pintype "passive"))
   )
-  (footprint "TestPoint:TestPoint_THTPad_D4.0mm_Drill2.0mm" (layer "F.Cu")
+  (footprint "TestPoint:TestPoint_THTPad_D5.0mm_Drill3.0mm" (layer "F.Cu")
     (at 92.75 112.557)
     (descr "THT pad as test Point, diameter 4.0mm, hole diameter 2.0mm")
@@
     (property "Sheetfile" "batteriedeckel.kicad_sch")
     (property "Sheetname" "")
-    (attr exclude_from_pos_files)
-    (fp_text reference "SW+" (at -4.612 -0.035) (layer "F.SilkS")
+    (attr exclude_from_pos_files exclude_from_bom)
+    (fp_text reference "SW+" (at 0 -2.898) (layer "F.SilkS")
       (effects (font (size 1 1) (thickness 0.15)))
     )
@@
       (effects (font (size 1 1) (thickness 0.15)))
     )
-    (fp_circle (center 0 0) (end 0 2.25) (layer "F.SilkS") (width 0.12) (fill none))
-    (fp_circle (center 0 0) (end 2.5 0) (layer "F.CrtYd") (width 0.05) (fill none))
-    (pad "1" thru_hole circle (at 0 0) (size 4 4) (drill 2) (layers *.Cu *.Mask)
+    (fp_circle (center 0 0) (end 2.5 0) (layer "F.SilkS") (width 0.12) (fill none))
+    (fp_circle (center 0 0) (end 3 0) (layer "F.CrtYd") (width 0.05) (fill none))
+    (pad "1" thru_hole circle (at 0 0) (size 5 5) (drill 3) (layers *.Cu *.Mask)
       (net 3 "/MODE") (pinfunction "1") (pintype "passive"))
   )
   (footprint "Connector_PinSocket_2.00mm:PinSocket_1x03_P2.00mm_Vertical_SMD_Pin1Left" (layer "F.Cu")
-    (at 100 100 -90)
+    (at 97.7 100)
     (descr "surface-mounted straight socket strip, 1x03, 2.00mm pitch, single row, style 1 (pin 1 left) (https://www.jayconsystems.com/fileuploader/download/download/?d=1&file=custom%2Fupload%2FFile-1375728122.pdf), script generated")
     (tags "Surface mounted socket strip SMD 1x03 2.00mm single row style1 pin1 left")
@@
     (property "Sheetname" "")
     (attr smd)
-    (fp_text reference "J1" (at -2.464 -5.664) (layer "F.SilkS")
-      (effects (font (size 1 1) (thickness 0.15)))
-    )
-    (fp_text value "Conn_01x03" (at 0 4.8 -90) (layer "F.Fab")
-      (effects (font (size 1 1) (thickness 0.15)))
-    )
-    (fp_text user "${REFERENCE}" (at 0 0) (layer "F.Fab")
+    (fp_text reference "J1" (at -2.464 -5.664 90) (layer "F.SilkS")
+      (effects (font (size 1 1) (thickness 0.15)))
+    )
+    (fp_text value "Conn_01x03" (at 0 4.8) (layer "F.Fab")
+      (effects (font (size 1 1) (thickness 0.15)))
+    )
+    (fp_text user "${REFERENCE}" (at 0 0 90) (layer "F.Fab")
       (effects (font (size 1 1) (thickness 0.15)))
     )
@@
     (fp_line (start -1.25 -2.675) (end -0.625 -3.3) (layer "F.Fab") (width 0.1))
     (fp_line (start 1.25 -3.3) (end 1.25 3.3) (layer "F.Fab") (width 0.1))
-    (pad "1" smd rect (at -1.6 -2 270) (size 2 0.9) (layers "F.Cu" "F.Paste" "F.Mask")
+    (pad "1" smd rect (at -1.6 -2) (size 2 0.9) (layers "F.Cu" "F.Paste" "F.Mask")
       (net 1 "/BAT+") (pinfunction "Pin_1") (pintype "passive"))
-    (pad "2" smd rect (at 1.6 0 270) (size 2 0.9) (layers "F.Cu" "F.Paste" "F.Mask")
+    (pad "2" smd rect (at 1.6 0) (size 2 0.9) (layers "F.Cu" "F.Paste" "F.Mask")
       (net 2 "/GND") (pinfunction "Pin_2") (pintype "passive"))
-    (pad "3" smd rect (at -1.6 2 270) (size 2 0.9) (layers "F.Cu" "F.Paste" "F.Mask")
+    (pad "3" smd rect (at -1.6 2) (size 2 0.9) (layers "F.Cu" "F.Paste" "F.Mask")
       (net 3 "/MODE") (pinfunction "Pin_3") (pintype "passive"))
     (model "${KICAD6_3DMODEL_DIR}/Connector_PinSocket_2.00mm.3dshapes/PinSocket_1x03_P2.00mm_Vertical_SMD_Pin1Left.wrl"
@@
     (effects (font (size 1 1) (thickness 0.2)))
   )
-  (segment (start 100 101.175) (end 100.175 101.175) (width 0.25) (layer "F.Cu") (net 2))
-  (segment (start 98 107.307) (end 98 98.825) (width 0.5) (layer "F.Cu") (net 3))
-  (segment (start 92.75 112.557) (end 98 107.307) (width 0.5) (layer "F.Cu") (net 3))
+  (segment (start 92.75 112.557) (end 96.266 109.041) (width 0.5) (layer "F.Cu") (net 3))
+  (segment (start 96.266 102.166) (end 96.1 102) (width 0.5) (layer "F.Cu") (net 3))
+  (segment (start 96.266 109.041) (end 96.266 102.166) (width 0.5) (layer "F.Cu") (net 3))
   (zone (net 1) (net_name "/BAT+") (layer "F.Cu") (hatch edge 0.508)
     (connect_pads yes (clearance 0.508))
@@
       (pts
         (xy 126.238 96.774)
-        (xy 103.124 96.774)
-        (xy 103.124 100.33)
-        (xy 101.092 100.33)
-        (xy 101.092 99.314)
-        (xy 99.06 99.314)
-        (xy 99.06 100.33)
+        (xy 102.108 96.774)
+        (xy 97.79 96.774)
+        (xy 97.79 100.33)
+        (xy 96.774 100.33)
         (xy 74.676 100.33)
         (xy 74.676 77.216)
@@
         (xy 74.676 123.444)
         (xy 74.676 100.584)
-        (xy 99.314 100.584)
-        (xy 99.314 99.568)
-        (xy 100.838 99.568)
-        (xy 100.838 100.584)
-        (xy 103.378 100.584)
-        (xy 103.378 97.028)
+        (xy 98.044 100.584)
+        (xy 98.044 97.028)
         (xy 126.238 97.028)
       )
