File: kicad/v5/led_buck_3a.kicad_sch (KiCad schematic)
At the start: 28 parts, among them J1 LED+, J2 LED-, J3 JST_B3B-PH-SM4-TB(LF)(SN), J4 Conn_01x05, Q1 BSC022N04LSATMA, U1 MAX16820ATT, U2 ATtiny1616-M

Commit message: save
Parts:
- added TP1, TP4: TestPoint, TestPoint:TestPoint_Pad_1.0x1.0mm, symbol Connector:TestPoint
- C1: footprint Capacitor_SMD:C_1210_3225Metric -> Capacitor_SMD:C_0805_2012Metric
Connections:
- net at U2.15 (PC0): now also TP4.1
- net at U2.16 (PC1): now also TP1.1
Changed lines of the file:
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@@
+    (stroke (width 0) (type default) (color 0 0 0 0))
+  )
+  (wire (pts (xy 191.135 68.58) (xy 201.93 68.58))
     (stroke (width 0) (type default) (color 0 0 0 0))
   )
@@
   )
   (wire (pts (xy 245.745 125.095) (xy 257.175 125.095))
+    (stroke (width 0) (type default) (color 0 0 0 0))
+  )
+  (wire (pts (xy 180.975 71.12) (xy 201.93 71.12))
     (stroke (width 0) (type default) (color 0 0 0 0))
   )
@@
     (pin "2")
   )
+  (symbol (lib_id "Connector:TestPoint") (at 191.135 68.58 90) (unit 1)
+    (in_bom yes) (on_board yes) (fields_autoplaced)
+    (property "Reference" "TP4" (id 0) (at 187.833 64.2452 90))
+    (property "Value" "TestPoint" (id 1) (at 187.833 66.7821 90))
+    (property "Footprint" "TestPoint:TestPoint_Pad_1.0x1.0mm" (id 2) (at 191.135 63.5 0)
+      (effects (font (size 1.27 1.27)) hide)
+    )
+    (property "Datasheet" "~" (id 3) (at 191.135 63.5 0)
+      (effects (font (size 1.27 1.27)) hide)
+    )
+    (pin "1")
+  )
   (symbol (lib_id "power:GND") (at 203.835 135.255 0) (unit 1)
     (in_bom yes) (on_board yes)
@@
       (effects (font (size 1.27 1.27)) (justify left))
     )
-    (property "Footprint" "Capacitor_SMD:C_1210_3225Metric" (id 2) (at 34.6202 69.85 0)
+    (property "Footprint" "Capacitor_SMD:C_0805_2012Metric" (id 2) (at 34.6202 69.85 0)
       (effects (font (size 1.27 1.27)) hide)
     )
@@
     (pin "7")
   )
+  (symbol (lib_id "Connector:TestPoint") (at 180.975 71.12 90) (unit 1)
+    (in_bom yes) (on_board yes) (fields_autoplaced)
+    (property "Reference" "TP1" (id 0) (at 177.673 66.7852 90))
+    (property "Value" "TestPoint" (id 1) (at 177.673 69.3221 90))
+    (property "Footprint" "TestPoint:TestPoint_Pad_1.0x1.0mm" (id 2) (at 180.975 66.04 0)
+      (effects (font (size 1.27 1.27)) hide)
+    )
+    (property "Datasheet" "~" (id 3) (at 180.975 66.04 0)
+      (effects (font (size 1.27 1.27)) hide)
+    )
+    (pin "1")
+  )
   (symbol (lib_id "Device:C") (at 107.315 93.98 0) (unit 1)
     (in_bom yes) (on_board yes)
@@
     )
     (path "/54d398f5-898b-4fd4-bf10-c22047e65de2"
-      (reference "C1") (unit 1) (value "22u0 / 25V") (footprint "Capacitor_SMD:C_1210_3225Metric")
+      (reference "C1") (unit 1) (value "22u0 / 25V") (footprint "Capacitor_SMD:C_0805_2012Metric")
     )
     (path "/520d5c7a-8c93-44c8-9867-1b7bcf9902fa"
@@
       (reference "R8") (unit 1) (value "470r") (footprint "Resistor_SMD:R_0805_2012Metric")
     )
+    (path "/9947e982-6573-4d47-be59-4873df21130f"
+      (reference "TP1") (unit 1) (value "TestPoint") (footprint "TestPoint:TestPoint_Pad_1.0x1.0mm")
+    )
+    (path "/062a424a-721b-4075-b935-eb8a71de4748"
+      (reference "TP4") (unit 1) (value "TestPoint") (footprint "TestPoint:TestPoint_Pad_1.0x1.0mm")
+    )
     (path "/966b5af4-8731-4826-b8cb-35f55786cf85"

Commit message: - Neues PCB V5.1 - Ädernungen an den Akkufach 3D Teilen - Firmware überarbeitet
Parts:
- removed C8: 4n70, Capacitor_SMD:C_0805_2012Metric, symbol Device:C
- removed R6: 10k0, Resistor_SMD:R_0805_2012Metric, symbol Device:R
- removed R7: CMFB103F3950FANT, Resistor_SMD:R_0805_2012Metric, symbol Device:R
- R3: value 82k5 -> 825k
- R4: value 6k81 -> 68k1
Connections:
- net TMESS: no longer names the net of U2.10 (PB4)
Other:
- note added: "History: - Remove NTC, use CPU internal Sensor - Change VMESS voltage divider to higher Values"
- moved on the sheet: C7, R3, R4
