File: kicad/v6/led_buck_3a.kicad_sch (KiCad schematic)
At the start: 27 parts, among them J1 LED+, J2 LED-, J3 JST_B3B-PH-SM4-TB(LF)(SN), J4 Conn_01x05, Q1 BSC022N04LSATMA, U1 MAX16820ATT, U2 ATtiny1616-M

Commit message: clean up
Parts:
- removed C3: DNP, Capacitor_SMD:C_0805_2012Metric, symbol Device:C
- removed J3: JST_B3B-PH-SM4-TB(LF)(SN), Connector_JST:JST_PH_B3B-PH-SM4-TB_1x03-1MP_P2.00mm_Vertical, symbol Connector_Generic:Conn_01x03
- added J3: Conn_02x03_Odd_Even, Connector_PinHeader_2.00mm:PinHeader_2x03_P2.00mm_Vertical_SMD, symbol Connector_Generic:Conn_02x03_Odd_Even
- C1: LCSC C90143 -> C45783
- Q1: value BSC022N04LSATMA -> BSC022N04LS6; LCSC C148266 -> C534307
- R1: value 0R070 -> 0R068; LCSC C76251 -> C534307
Connections:
- net GND: now also J3.3 (Pin_3), J3.4 (Pin_4)
- net MODE: now also J3.2 (Pin_2), J3.5 (Pin_5)
- net VCC: now also J3.1 (Pin_1), J3.6 (Pin_6)
Other:
- moved on the sheet: R2
